File: hardware/POWER/v1.0/husb238.kicad_sch (KiCad schematic)
At the start: 8 parts, among them U1 HUSB238, U3 CSD25402Q3A

Commit message: 硬件1.0版本更新
Connections:
- net VBUS_IN: now also U3.5 (S); no longer U3.1 (D), U3.2 (D), U3.3 (D)
- net VBUS_OUT: now also U3.1 (D), U3.2 (D), U3.3 (D); no longer U3.5 (S)
Other:
- moved on the sheet: U3
Changed lines of the file:
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@@
 	(symbol
 		(lib_id "Transistor_FET:CSD25402Q3A")
-		(at 152.4 69.85 90)
+		(at 152.4 69.85 270)
+		(mirror x)
 		(unit 1)
 		(exclude_from_sim no)
@@
 		(on_board yes)
 		(dnp no)
-		(fields_autoplaced yes)
 		(property "Reference" "U3"
 			(at 152.4 60.96 90)
@@
 		)
 		(property "Footprint" "Package_SON:VSON-8_3.3x3.3mm_P0.65mm_NexFET"
-			(at 157.099 39.497 0)
+			(at 147.701 39.497 0)
 			(effects
 				(font
@@
 		)
 		(property "Datasheet" "https://www.ti.com/lit/ds/symlink/csd25402q3a.pdf"
-			(at 154.813 38.735 0)
+			(at 149.987 38.735 0)
 			(effects
 				(font
